File: stm32f4-discovery-breakout-v2.sch (EAGLE design)
At the start: 5 parts

Commit message: Fixed up version numbers.
Parts:
- J1, J2, J3, J4: value M25LOCK_LONGPADS -> (none)
- renumbered JP1 to J1, JP2 to J2, JP3 to J3, JP4 to J4
